Commit message: gps files added

File: moborobo/description/robot.udrf.xacro (robot description, xacro)
@@ -5,4 +5,6 @@
         <xacro:include filename="camera.xacro"/>
         <xacro:include filename="stereo_camera.xacro"/>
+        <xacro:include filename="gps.xacro"/>
+        <xacro:include filename="imu.xacro"/>
         <xacro:include filename="$(find moborobo)/urdf/RS-16.urdf.xacro"/>
     </robot>

File: moborobo/description/stereo_camera.xacro (robot description, xacro)
@@ -4,5 +4,5 @@
         <parent link="base_link"/>
         <child link="stereo_camera_link"/>
-        <origin xyz="-0.21 0 0.51" rpy="0 0 0"/>
+        <origin xyz="-0.20 0 0.51" rpy="0 0 ${pi}"/>
     </joint>
     <link name="stereo_camera_link">
@@ -25,5 +25,5 @@
       <parent link="stereo_camera_link"/>
       <child link="stereo_left_camera_frame"/>
-      <origin xyz="0 -0.07 0" rpy="0 0 0" />
+      <origin xyz="0 0.07 0" rpy="0 0 0" />
     </joint>
     <link name="stereo_left_camera_frame" />
@@ -38,5 +38,5 @@
       <parent link="stereo_camera_link"/>
       <child link="stereo_right_camera_frame"/>
-      <origin xyz="0 0.07 0" rpy="0 0 0" />
+      <origin xyz="0 -0.07 0" rpy="0 0 0" />
     </joint>
     <link name="stereo_right_camera_frame" />
